File: TR-808-Clone.sch (KiCad schematic (older format))
At the start: 456 parts, among them Q45 MMBT3904, Q46 MMBT3906

Commit message: starting manual annoation to match original 808 schematic. Snare Drum annoation done
Parts:
- C51: renamed from C?; value 47μ -> 0.47μ
- C53: renamed from C?; value 0.1μ -> 0.001μ
- VR7: value 100K -> 100K(A)
- VR8: value 100K -> 100K(B)
- VR9: value 10K -> 10K(B)
- gave numbers to parts that had none: 46

Commit message: bass drum annoated
Parts:
- added R164: 47K, symbol R_US
- VR4: value POT_US -> 100K(A)
- VR5: value 10K -> 10K(C)
- VR6: value 500K -> 500K(B)
- gave numbers to parts that had none: 45
Connections:
- wire segments 894 -> 1186
Other:
- note added: "A: LOG TAPER\nB: LINEAR TAPER\nC: ANTI-LOG TAPER"
- moved on the sheet: C41, C42, R166, R169, R173

Commit message: low tom/conga annotated
Parts:
- R234: renamed from R?; value 820K -> 47K
- VR10: renamed from VR?; value 100K -> 100K(A)
- VR11: renamed from VR?; value 500K -> 500(B)
- VR?: value 100K -> 100K(A)
- gave numbers to parts that had none: 46
Connections:
- wire segments 1186 -> 1185
Other:
- note added: "**"
- moved on the sheet: C83, R227

Commit message: mid tom/conga and hi tom/conga annotated
Parts:
- R263, R290: renamed from R?; value 820K -> 47K
- VR12, VR14: renamed from VR?; value 100K -> 100K(A)
- VR13, VR15: renamed from VR?; value 500K -> 500(B)
- VR? (x2): value 100K -> 100K(B)
- gave numbers to parts that had none: 91
Connections:
- net labels added: HT_TRIG, MT_TRIG
Other:
- moved on the sheet: C97, R256, R266, R283

Commit message: rim shot/claves annotated
Parts:
- added R306: 22K, symbol R_US
- R324: value VALUE -> 220K
- VR16: renamed from VR?; value 100K -> 100K(A)
- gave numbers to parts that had none: 62
Connections:
- wire segments 1185 -> 895
Other:
- moved on the sheet: C111, C117, C119, C126, C153, D62, R301, R302, R307, R308, R326, R330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

Commit message: clap/maracas annotated
Parts:
- added unit 2 of U22
- added U?: 4558, symbol TL072-
- C128, C129: renamed from C?; value 0.047μ -> 0.0047μ
- TM3: renamed from VR?; value 10K -> 10K(B)
- U23: renamed from U?; value LM339- -> LM339
- VR17: renamed from VR?; value 100K -> 100K(A)
- gave numbers to parts that had none: 95
Connections:
- wire segments 895 -> 1191
- no-connect marks 10 -> 16
Other:
- moved on the sheet: C146

Commit message: cowbell annotated
Changed lines of the file:
@@
 Text GLabel 5775 12375 2    60   Input ~ 0
 WHITE_NOISE
-Text Notes 825  6425 0    100  ~ 0
+Text Notes 825  6550 0    200  ~ 40
 SNARE DRUM\n
 $Comp
@@
 Text Notes 8075 5075 0    60   ~ 12
 BD\nLEVEL
-Text Notes 825  875  0    100  ~ 0
+Text Notes 800  1025 0    200  ~ 40
 BASS DRUM\n
 $Comp
@@
 Text Notes 17200 4775 0    60   ~ 12
 LT/LC\nREVERB\n
-Text Notes 10850 875  0    100  ~ 0
+Text Notes 10875 1000 0    200  ~ 40
 LOW TOM/CONGA
 $Comp
@@
 Text Notes 27000 4775 0    60   ~ 12
 MT/MC\nREVERB\n
-Text Notes 20650 875  0    100  ~ 0
+Text Notes 20675 1000 0    200  ~ 40
 MID TOM/CONGA
 $Comp
@@
 Text Notes 36850 4775 0    60   ~ 12
 HT/HC\nREVERB\n
-Text Notes 30500 875  0    100  ~ 0
+Text Notes 30500 1000 0    200  ~ 40
 HI TOM/CONGA
 Text Notes 23725 2350 0    60   ~ 0
@@
 	1    0    0    -1
 $EndComp
-Text Notes 825  13425 0    100  ~ 0
+Text Notes 800  13525 0    200  ~ 40
 CLAP/MARACAS
 $Comp
@@
 Wire Notes Line
 	10775 13525 10775 6250
-Text Notes 10875 6475 0    100  ~ 0
+Text Notes 10850 6550 0    200  ~ 40
 RIM SHOT/CLAVES\n
 Text Notes 29425 29400 0    200  ~ 40

Commit message: cymbal annotated
Connections:
- net labels added: COMMON_TRIG
- net labels removed: ACCENT
Changed lines of the file:
@@
 Text GLabel 1250 8075 0    60   Input ~ 0
 SD_TRIG
-Text GLabel 1250 7275 0    60   Input ~ 0
-ACCENT
+Text GLabel 1500 7275 0    60   Input ~ 0
+COMMON_TRIG
 $Comp
 L R_US R199
@@
 Text GLabel 1475 3400 0    60   Input ~ 0
 BD_TRIG
-Text GLabel 1325 2375 0    60   Input ~ 0
-ACCENT
+Text GLabel 1675 2375 0    60   Input ~ 0
+COMMON_TRIG
 $Comp
 L TL072- U15
@@
 Text GLabel 11300 2950 0    60   Input ~ 0
 LT_TRIG
-Text GLabel 11300 2150 0    60   Input ~ 0
-ACCENT
+Text GLabel 11650 2150 0    60   Input ~ 0
+COMMON_TRIG
 $Comp
 L R_US R215
@@
 Text GLabel 21100 2950 0    60   Input ~ 0
 MT_TRIG
-Text GLabel 21100 2150 0    60   Input ~ 0
-ACCENT
+Text GLabel 21500 2150 0    60   Input ~ 0
+COMMON_TRIG
 $Comp
 L R_US R251
@@
 Text GLabel 30950 2950 0    60   Input ~ 0
 HT_TRIG
-Text GLabel 30950 2150 0    60   Input ~ 0
-ACCENT
+Text GLabel 31225 2150 0    60   Input ~ 0
+COMMON_TRIG
 $Comp
 L R_US R270
@@
 Text GLabel 1425 15200 0    60   Input ~ 0
 CP_TRIG
-Text GLabel 1400 14600 0    60   Input ~ 0
-ACCENT
+Text GLabel 1575 14600 0    60   Input ~ 0
+COMMON_TRIG
 Text Notes 2625 16225 0    60   ~ 0
 CP
@@
 RS_TRIG
 Text GLabel 11700 7100 0    60   Input ~ 0
-ACCENT
+COMMON_TRIG
 $Comp
 L D D61
@@
 	2275 7275 2275 7700
 Wire Wire Line
-	1250 7275 1875 7275
+	1500 7275 1875 7275
 Wire Wire Line
 	1875 7275 2275 7275
@@
 	2350 2375 2350 2800
 Wire Wire Line
-	1325 2375 1950 2375
+	1675 2375 1950 2375
 Wire Wire Line
 	1950 2375 2350 2375
@@
 	12325 2150 12325 2575
 Wire Wire Line
-	11300 2150 11925 2150
+	11650 2150 11925 2150
 Wire Wire Line
 	11925 2150 12325 2150
@@
 	22125 2150 22125 2575
 Wire Wire Line
-	21100 2150 21725 2150
+	21500 2150 21725 2150
 Wire Wire Line
 	21725 2150 22125 2150
@@
 	31975 2150 31975 2575
 Wire Wire Line
-	30950 2150 31575 2150
+	31225 2150 31575 2150
 Wire Wire Line
 	31575 2150 31975 2150
@@
 	2450 14600 2450 15025
 Wire Wire Line
-	1400 14600 1900 14600
+	1575 14600 1900 14600
 Wire Wire Line
 	1900 14600 2450 14600
@@
 F3 "-V" I L 19525 16250 60
 F4 "GND" I L 19525 16375 60
-F5 "ACCENT" I L 19525 16500 60
+F5 "COMMON_TRIG" I L 19525 16500 60
 F6 "CB_TRIG" I L 19525 16600 60
 F7 "CB" O L 19525 16700 60
