File: BA662.sch (KiCad schematic (older format))
At the start: 11 parts, among them Q1-1 PMP4201, Q2-1 PMP4201, Q3-1 PMP5201, Q4-1 PMP5201, Q5-1 PMP5201, Q6-1 PMP4201, Q7-1 PMP4201, Q8-1 PMP5201, Q9-1 PMP4201

Commit message: Sync LED control pins added, tom clipping diodes changed to BAT54 with series resistor
Other:
- note added: "Discrete BA662 clone\nfrom Open Music Labs"
- note added: "http://www.openmusiclabs.com/"
- moved on the sheet: Q1-1A, Q1-1B, Q2-1A, Q2-1B, Q3-1A, Q3-1B, Q4-1A, Q4-1B, Q5-1A, Q5-1B, Q6-1A, Q6-1B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

Commit message: assigning footprints before importing updated netlist into pcbnew
Parts:
- R179, R328: footprint (none) -> MyModules:SM0603-R-JRL
Changed lines of the file:
@@
 F 0 "R179" V 6355 4050 50  0000 C CNN
 F 1 "47K" V 6195 4050 50  0000 C CNN
-F 2 "" H 6275 4050 60  0000 C CNN
+F 2 "MyModules:SM0603-R-JRL" H 6275 4050 60  0001 C CNN
 F 3 "" H 6275 4050 60  0000 C CNN
 	1    6275 4050
@@
 F 0 "R328" V 7405 3575 50  0000 C CNN
 F 1 "10K" V 7245 3575 50  0000 C CNN
-F 2 "" H 7325 3575 60  0000 C CNN
+F 2 "MyModules:SM0603-R-JRL" H 7325 3575 60  0001 C CNN
 F 3 "" H 7325 3575 60  0000 C CNN
 	1    7325 3575
