File: back_panel.kicad_pcb (KiCad board)
At the start: 4 copper layers, 300 x 105 mm, 48 parts, among them P1 CONN_02X05, P2 CONN_01X08, P3 CONN_02X10, P6 CONN_01X03, P7 CONN_02X03, U35 R-78E5.0-0.5

Commit message: almost done first version of back panel
Parts:
- removed P2: CONN_01X08, MyModules:Molex_522710479_8_FFC
- added G***: LOGO, LOGO, B.Cu at (350.4, 132.2)
- added REF**: pad_3_mm, pad_3_mm, B.Cu at (222.7, 75.2)
- added REF**: pad_3_mm, pad_3_mm, B.Cu at (243.7, 68.2)
- added REF**: pad_3_mm, pad_3_mm, B.Cu at (222.7, 68.2)
- added REF**: pad_3_mm, pad_3_mm, B.Cu at (208.7, 68.2)
- added REF**: pad_3_mm, pad_3_mm, B.Cu at (201.7, 68.2)
- added REF**: pad_3_mm, pad_3_mm, B.Cu at (194.7, 68.2)
- added REF**: pad_3_mm, pad_3_mm, B.Cu at (173.7, 68.2)
- added REF**: pad_3_mm, pad_3_mm, B.Cu at (194.7, 82.2)
- added REF**: pad_3_mm, pad_3_mm, B.Cu at (229.7, 82.2)
- added REF**: pad_3_mm, pad_3_mm, B.Cu at (250.7, 82.2)
- added REF**: pad_3_mm, pad_3_mm, B.Cu at (334.6, 89.2)
- added REF**: pad_3_mm, pad_3_mm, B.Cu at (75.7, 54.1)
- added REF**: pad_3_mm, pad_3_mm, B.Cu at (285.6, 89.2)
- added REF**: pad_3_mm, pad_3_mm, B.Cu at (278.6, 89.2)
- added REF**: pad_3_mm, pad_3_mm, B.Cu at (278.6, 82.2)
- added REF**: pad_3_mm, pad_3_mm, B.Cu at (285.6, 82.2)
- added REF**: pad_3_mm, pad_3_mm, B.Cu at (292.6, 82.2)
- added REF**: pad_3_mm, pad_3_mm, B.Cu at (292.6, 75.2)
- added REF**: pad_3_mm, pad_3_mm, B.Cu at (292.6, 68.2)
- added REF**: pad_3_mm, pad_3_mm, B.Cu at (320.6, 82.2)
- added REF**: pad_3_mm, pad_3_mm, B.Cu at (355.6, 103.2)
- added REF**: pad_3_mm, pad_3_mm, B.Cu at (355.6, 96.2)
- added REF**: pad_3_mm, pad_3_mm, B.Cu at (180.7, 82.2)
- added REF**: pad_3_mm, pad_3_mm, B.Cu at (362.6, 96.2)
- added REF**: pad_3_mm, pad_3_mm, B.Cu at (362.6, 89.2)
- added REF**: pad_3_mm, pad_3_mm, B.Cu at (348.6, 89.2)
- added REF**: pad_3_mm, pad_3_mm, B.Cu at (348.6, 82.2)
- added REF**: pad_3_mm, pad_3_mm, B.Cu at (285.6, 96.2)
- added REF**: pad_3_mm, pad_3_mm, B.Cu at (215.7, 89.2)
- added REF**: pad_3_mm, pad_3_mm, B.Cu at (208.7, 89.2)
- added REF**: pad_3_mm, pad_3_mm, B.Cu at (187.7, 82.2)
- added REF**: pad_3_mm, pad_3_mm, B.Cu at (166.7, 75.2)
- added REF**: pad_3_mm, pad_3_mm, B.Cu at (362.6, 75.2)
- added REF**: pad_3_mm, pad_3_mm, B.Cu at (320.6, 68.2)
- added REF**: pad_3_mm, pad_3_mm, B.Cu at (355.6, 75.2)
- added REF**: pad_3_mm, pad_3_mm, B.Cu at (348.6, 75.2)
- added REF**: pad_3_mm, pad_3_mm, B.Cu at (320.6, 75.2)
- added REF**: pad_3_mm, pad_3_mm, B.Cu at (313.6, 75.2)
- added REF**: pad_3_mm, pad_3_mm, B.Cu at (306.6, 75.2)
- added REF**: pad_3_mm, pad_3_mm, B.Cu at (264.6, 75.2)
- added REF**: pad_3_mm, pad_3_mm, B.Cu at (257.6, 75.2)
- added REF**: pad_3_mm, pad_3_mm, B.Cu at (250.7, 75.2)
- added REF**: pad_3_mm, pad_3_mm, B.Cu at (215.7, 75.2)
- added REF**: pad_3_mm, pad_3_mm, B.Cu at (208.7, 75.2)
- added REF**: pad_3_mm, pad_3_mm, B.Cu at (327.6, 96.2)
- added REF**: pad_3_mm, pad_3_mm, B.Cu at (187.7, 75.2)
- added REF**: pad_3_mm, pad_3_mm, B.Cu at (103.7, 61.1)
- added REF**: pad_3_mm, pad_3_mm, B.Cu at (138.7, 68.2)
- added REF**: pad_3_mm, pad_3_mm, B.Cu at (145.7, 61.1)
- added REF**: pad_3_mm, pad_3_mm, B.Cu at (166.7, 61.1)
- added REF**: pad_3_mm, pad_3_mm, B.Cu at (187.7, 61.1)
- added REF**: pad_3_mm, pad_3_mm, B.Cu at (222.7, 61.1)
- added REF**: pad_3_mm, pad_3_mm, B.Cu at (243.7, 61.1)
- added REF**: pad_3_mm, pad_3_mm, B.Cu at (264.6, 61.1)
- added REF**: pad_3_mm, pad_3_mm, B.Cu at (285.6, 61.1)
- added REF**: pad_3_mm, pad_3_mm, B.Cu at (334.6, 96.2)
- added REF**: pad_3_mm, pad_3_mm, B.Cu at (306.6, 61.1)
- added REF**: pad_3_mm, pad_3_mm, B.Cu at (327.6, 61.1)
- added REF**: pad_3_mm, pad_3_mm, B.Cu at (355.6, 61.1)
- added REF**: pad_3_mm, pad_3_mm, B.Cu at (362.6, 54.1)
- added REF**: pad_3_mm, pad_3_mm, B.Cu at (348.6, 54.1)
- added REF**: pad_3_mm, pad_3_mm, B.Cu at (334.6, 54.1)
- added REF**: pad_3_mm, pad_3_mm, B.Cu at (306.6, 54.1)
- added REF**: pad_3_mm, pad_3_mm, B.Cu at (292.6, 54.1)
- added REF**: pad_3_mm, pad_3_mm, B.Cu at (285.6, 54.1)
- added REF**: pad_3_mm, pad_3_mm, B.Cu at (278.6, 54.1)
- added REF**: pad_3_mm, pad_3_mm, B.Cu at (334.6, 82.2)
- added REF**: pad_3_mm, pad_3_mm, B.Cu at (264.6, 54.1)
- added REF**: pad_3_mm, pad_3_mm, B.Cu at (250.7, 54.1)
- added REF**: pad_3_mm, pad_3_mm, B.Cu at (236.7, 54.1)
- added REF**: pad_3_mm, pad_3_mm, B.Cu at (215.7, 54.1)
- added REF**: pad_3_mm, pad_3_mm, B.Cu at (194.7, 54.1)
- added REF**: pad_3_mm, pad_3_mm, B.Cu at (173.7, 54.1)
- added REF**: pad_3_mm, pad_3_mm, B.Cu at (159.7, 54.1)
- added REF**: pad_3_mm, pad_3_mm, B.Cu at (138.7, 54.1)
- added REF**: pad_3_mm, pad_3_mm, B.Cu at (159.7, 75.2)
- added REF**: pad_3_mm, pad_3_mm, B.Cu at (117.7, 54.1)
- added REF**: pad_3_mm, pad_3_mm, B.Cu at (334.6, 68.2)
- added REF**: pad_3_mm, pad_3_mm, B.Cu at (103.7, 54.1)
- added REF**: pad_3_mm, pad_3_mm, B.Cu at (89.7, 54.1)
- added REF**: pad_3_mm, pad_3_mm, B.Cu at (278.6, 68.2)
- added SNAP-HOLE-0.125-INCH: VAL**, MyModules:SNAP_HOLE_0.125_INCH, F.Cu at (185.9, 38.2)
- added SNAP-HOLE-0.125-INCH: VAL**, MyModules:SNAP_HOLE_0.125_INCH, F.Cu at (176.7, 43.6)
- added SNAP-HOLE-0.125-INCH: VAL**, MyModules:SNAP_HOLE_0.125_INCH, F.Cu at (180.9, 40.1)
- added SNAP-HOLE-0.125-INCH: VAL**, MyModules:SNAP_HOLE_0.125_INCH, F.Cu at (176.2, 40.1)
- added SNAP-HOLE-0.125-INCH: VAL**, MyModules:SNAP_HOLE_0.125_INCH, F.Cu at (172.4, 40.6)
- added SNAP-HOLE-0.125-INCH: VAL**, MyModules:SNAP_HOLE_0.125_INCH, F.Cu at (167.7, 40.6)
- G***: moved to F.Cu
- moved G*** 4.50 mm to (179.9, 109.9)
- turned G*** to 0 degrees
Routing:
- net (no net): track 0.00 -> 3248.3 mm
Other:
- outline, holes or cut-outs redrawn
- copper layers 4 -> 2
- rule pad_to_mask_clearance: 0.025 -> 0
- board text added: "!"
- board text added: "880 back panel r1.0 09/2018"
- board text added: "ISP"
- board text added: "SYSTEM80 INC. TORONTO CANADA"
- board text added: "TRIGGER 2 LEVEL"
- board text added: "systme80.net"

Commit message: back panel design almost done
Parts:
- removed the G*** at (179.9, 109.9)
- removed REF***: OSHW-Symbol_6.7x6mm_SilkScreen, Symbols:OSHW-Symbol_6.7x6mm_SilkScreen
- added G***: LOGO, Logo_copper_OSHW_6x6mm, B.Cu at (73.7, 127.2)
- added G***: LOGO, LOGO, B.Cu at (350.4, 145.2)
- added G***: LOGO, LOGO, B.Cu at (191.9, 152.2)
- added G***: LOGO, LOGO, B.Cu at (180.2, 114.7)
- moved REF** 39.6 mm to (257.6, 68.2)
- moved G*** 5.26 mm to (350.6, 126.9)
Routing:
- net (no net): track 3248.3 -> 3250.5 mm
Other:
- board text removed: "SYSTEM80 INC. TORONTO CANADA"
- board text removed: "systme80.net"

Commit message: production PCBs ordered, working on manual
Parts:
- removed the G*** at (191.9, 152.2)
- removed ISP1: CONN_02X03, w_conn_strip:vasch_strip_3x2
- removed P1: CONN_02X05, Pin_Headers:Pin_Header_Straight_2x05
- removed P3: CONN_02X10, w_conn_strip:vasch_strip_10x2
- removed P6 (x2): CONN_01X03, Pin_Headers:Pin_Header_Straight_1x03
- removed P7: CONN_02X03, DIY:PIN_ARRAY_3X2
- removed TM1, TM2: 200K(B), MyModules:TC33X-2
- removed TM3: 10K(B), MyModules:TC33X-2
- removed TM4: 20K(B), MyModules:TC33X-2
- removed TP13, TP7: TEST_POINT, MyModules:TEST_POINT_LOOP_4592
- removed TP17: CONN_1, MyModules:TEST POINT
- removed TP18, TP19: CONN_1, MyModules:TEST_POINT_LOOP_4592
- removed TP6: TEST_POINT, MyModules:TEST_POINT_5000_SERIES
- removed U35: R-78E5.0-0.5, MyModules:R-78E-0.5

Commit message: added operation rerference page to manual, added a couple of notes about clap reverb changes
Parts:
- added SNAP-HOLE-0.125-INCH: VAL**, MyModules:SNAP_HOLE_0.125_INCH, F.Cu at (297.1, 114.2)

Commit message: updates to back panel
Routing:
- net (no net): track 3250.5 -> 3260.3 mm
