File: back_panel.kicad_pcb (KiCad board)
At the start: 2 copper layers, 300 x 105 mm, 120 parts

Commit message: update manual
Parts:
- added G***: LOGO, LOGO, F.Cu at (311.9, 84.2)
- moved G*** 41.5 mm to (350.9, 105.7)
Other:
- board text added: "880 back panel r1.1 11/2018"
- board text removed: "880 back panel r1.0 09/2018"
