File: step_switch_board/step_switch_board.sch (KiCad schematic (older format))
At the start: 75 parts, among them P3 CONN_01X08, SW23 STEP1, SW24 STEP2, SW25 STEP3, SW26 STEP4, SW27 STEP5, SW28 STEP6, SW29 STEP7, SW30 STEP8, SW31 STEP9, SW32 STEP10, SW33 STEP11, SW34 STEP12, SW35 STEP13, SW36 STEP14, SW37 STEP15, SW38 STEP16, U38 74HC165, U39 74HC165, U40 74AC595, U41 74AC595

Commit message: started panel layout in Inkscape
Other:
- note added: "SPI SWITCH LATCH BYTE 3"
- note added: "SPI SWITCH LATCH BYTE 4"
- note removed: "SPI SWITCH LATCH 1"
- note removed: "SPI SWITCH LATCH 2"
Changed lines of the file:
@@
 LIBS:valves
 LIBS:MySynthParts
+LIBS:step_switch_board-cache
 EELAYER 25 0
 EELAYER END
@@
 NoConn ~ 13050 7075
 NoConn ~ 1475 4175
-Text Notes 1025 3750 0    60   ~ 0
-SPI SWITCH LATCH 1
-Text Notes 5550 3725 0    60   ~ 0
-SPI SWITCH LATCH 2
+Text Notes 850  3875 0    60   ~ 0
+SPI SWITCH LATCH BYTE 4
+Text Notes 5350 3875 0    60   ~ 0
+SPI SWITCH LATCH BYTE 3
 $Comp
 L CONN_01X08 P3

Commit message: added larger bypass caps to switch board, adding coupling caps to critical op amps
Parts:
- added C196, C197: 10µ, Capacitors_SMD:C_1206, symbol C_US
Connections:
- net +5V: now also C196.1, C197.1
- net GND: now also C196.2, C197.2
Changed lines of the file:
@@
 L 5V #PWR033
 U 1 1 56BE19E9
-P 1825 7025
-F 0 "#PWR033" H 1825 6875 50  0001 C CNN
-F 1 "5V" H 1825 7200 50  0000 C CNN
-F 2 "" H 1825 7025 60  0000 C CNN
-F 3 "" H 1825 7025 60  0000 C CNN
-	1    1825 7025
+P 1825 6700
+F 0 "#PWR033" H 1825 6550 50  0001 C CNN
+F 1 "5V" H 1825 6875 50  0000 C CNN
+F 2 "" H 1825 6700 60  0000 C CNN
+F 3 "" H 1825 6700 60  0000 C CNN
+	1    1825 6700
 	1    0    0    -1
 $EndComp
 Wire Wire Line
-	1825 7025 1825 7075
+	1825 6700 1825 7075
 Wire Wire Line
 	1825 7075 1875 7075
@@
 Text GLabel 1875 7675 0    50   Input ~ 0
 SPI_LED_DATA
+$Comp
+L C_US C197
+U 1 1 5AEB6DD9
+P 1250 6925
+F 0 "C197" H 1300 7025 50  0000 L CNN
+F 1 "10µ" H 1300 6825 50  0000 L CNN
+F 2 "Capacitors_SMD:C_1206" H 1250 6925 60  0000 C CNN
+F 3 "~" H 1250 6925 60  0000 C CNN
+	1    1250 6925
+	1    0    0    -1
+$EndComp
+$Comp
+L GND_E #PWR?
+U 1 1 5AEB7B3E
+P 1250 7200
+F 0 "#PWR?" V 1250 7200 30  0001 C CNN
+F 1 "GND_E" H 1250 7130 30  0001 C CNN
+F 2 "~" H 1250 7200 60  0000 C CNN
+F 3 "~" H 1250 7200 60  0000 C CNN
+	1    1250 7200
+	1    0    0    -1
+$EndComp
+Wire Wire Line
+	1250 7125 1250 7200
+Wire Wire Line
+	900  6725 1825 6725
+Connection ~ 1825 6725
+$Comp
+L C_US C196
+U 1 1 5AEB84B6
+P 900 6925
+F 0 "C196" H 950 7025 50  0000 L CNN
+F 1 "10µ" H 950 6825 50  0000 L CNN
+F 2 "Capacitors_SMD:C_1206" H 900 6925 60  0000 C CNN
+F 3 "~" H 900 6925 60  0000 C CNN
+	1    900  6925
+	1    0    0    -1
+$EndComp
+Connection ~ 1250 6725
+Wire Wire Line
+	1250 7150 900  7150
+Wire Wire Line
+	900  7150 900  7125
+Connection ~ 1250 7150
 $EndSCHEMATC
